File: hardware/protovolt/protovolt.kicad_sch (KiCad schematic)
At the start: 2 parts, among them J1 USB_C_Receptacle_USB2.0_16P, U1 CH224K

Commit message: finish demo schematic
Parts:
- removed J1: USB_C_Receptacle_USB2.0_16P, symbol Connector:USB_C_Receptacle_USB2.0_16P
- removed U1: CH224K, Package_SO:SSOP-10-1EP_3.9x4.9mm_P1mm_EP2.1x3.3mm, symbol Interface_USB:CH224K
Changed lines of the file:
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@@
 	(generator_version "8.0")
 	(paper "A3")
-	(symbol
-		(lib_id "Connector:USB_C_Receptacle_USB2.0_16P")
-		(at 182.88 143.51 0)
-		(unit 1)
-		(exclude_from_sim no)
-		(in_bom yes)
-		(on_board yes)
-		(dnp no)
-		(fields_autoplaced yes)
-		(property "Reference" "J1"
-			(at 182.88 120.65 0)
-			(effects
-				(font
-					(size 1.27 1.27)
-				)
-			)
-		)
-		(property "Value" "USB_C_Receptacle_USB2.0_16P"
-			(at 182.88 123.19 0)
-			(effects
-				(font
-					(size 1.27 1.27)
-				)
-			)
-		)
-		(property "Footprint" ""
-			(at 186.69 143.51 0)
-			(effects
-				(font
-					(size 1.27 1.27)
-				)
-				(hide yes)
-			)
-		)
-		(property "Datasheet" "https://www.usb.org/sites/default/files/documents/usb_type-c.zip"
-			(at 186.69 143.51 0)
-			(effects
-				(font
-					(size 1.27 1.27)
-				)
-				(hide yes)
-			)
-		)
-		(property "Description" "USB 2.0-only 16P Type-C Receptacle connector"
-			(at 182.88 143.51 0)
-			(effects
-				(font
-					(size 1.27 1.27)
-				)
-				(hide yes)
-			)
-		)
-		(property "LCSC" ""
-			(at 182.88 143.51 0)
-			(effects
-				(font
-					(size 1.27 1.27)
-				)
-				(hide yes)
-			)
-		)
-		(pin "B8"
-		)
-		(pin "B12"
-		)
-		(pin "B1"
-		)
-		(pin "A4"
-		)
-		(pin "S1"
-		)
-		(pin "A12"
-		)
-		(pin "A8"
-		)
-		(pin "B4"
-		)
-		(pin "A9"
-		)
-		(pin "A7"
-		)
-		(pin "B5"
-		)
-		(pin "A5"
-		)
-		(pin "B6"
-		)
-		(pin "B7"
-		)
-		(pin "A6"
-		)
-		(pin "B9"
-		)
-		(pin "A1"
-		)
-		(instances
-			(project ""
-				(path "/ea7037dc-92a2-412b-b904-472cbab72219"
-					(reference "J1")
-					(unit 1)
-				)
-			)
-		)
-	)
-	(symbol
-		(lib_id "Interface_USB:CH224K")
-		(at 102.87 129.54 0)
-		(unit 1)
-		(exclude_from_sim no)
-		(in_bom yes)
-		(on_board yes)
-		(dnp no)
-		(fields_autoplaced yes)
-		(property "Reference" "U1"
-			(at 105.0641 139.7 0)
-			(effects
-				(font
-					(size 1.27 1.27)
-				)
-				(justify left)
-			)
-		)
-		(property "Value" "CH224K"
-			(at 105.0641 142.24 0)
-			(effects
-				(font
-					(size 1.27 1.27)
-				)
-				(justify left)
-			)
-		)
-		(property "Footprint" "Package_SO:SSOP-10-1EP_3.9x4.9mm_P1mm_EP2.1x3.3mm"
-			(at 102.87 153.67 0)
-			(effects
-				(font
-					(size 1.27 1.27)
-				)
-				(hide yes)
-			)
-		)
-		(property "Datasheet" "https://www.wch.cn/downloads/file/301.html"
-			(at 102.87 115.57 0)
-			(effects
-				(font
-					(size 1.27 1.27)
-				)
-				(hide yes)
-			)
-		)
-		(property "Description" "100W USB Type-C PD3.0/2.0, BC1.2 Sink Controller, SSOP-10"
-			(at 102.87 129.54 0)
-			(effects
-				(font
-					(size 1.27 1.27)
-				)
-				(hide yes)
-			)
-		)
-		(property "LCSC" ""
-			(at 102.87 129.54 0)
-			(effects
-				(font
-					(size 1.27 1.27)
-				)
-				(hide yes)
-			)
-		)
-		(pin "5"
-		)
-		(pin "10"
-		)
-		(pin "8"
-		)
-		(pin "1"
-		)
-		(pin "7"
-		)
-		(pin "4"
-		)
-		(pin "3"
-		)
-		(pin "11"
-		)
-		(pin "6"
-		)
-		(pin "2"
-		)
-		(pin "9"
-		)
-		(instances
-			(project ""
-				(path "/ea7037dc-92a2-412b-b904-472cbab72219"
-					(reference "U1")
-					(unit 1)
-				)
-			)
-		)
-	)
 	(sheet
 		(at 153.67 71.12)
@@
 			(project "protovolt"
 				(path "/ea7037dc-92a2-412b-b904-472cbab72219"
-					(page "2")
+					(page "3")
 				)
 			)
