File: hardware/protovolt/output_A.kicad_sch (KiCad schematic)
At the start: 76 parts, among them J1 Conn_01x03, J10 Conn_02x03_Odd_Even, J2 Conn_01x03, J3 Conn_01x03, J4 Conn_01x03, J5 Conn_01x03, J6 Conn_01x03, J7 Conn_01x03, J8 Conn_01x03, J9 Conn_02x03_Odd_Even, Q1 BSC0702LS, Q2 BSC0702LS, Q3 BSC0702LS, Q4 BSC0702LS, Q5 BSC0702LS, U1 INA226, U2 LM51772RHAR

Commit message: finalize DRU & PCB
Parts:
- Q1, Q2, Q3, Q4, Q5: footprint Package_TO_SOT_SMD:TDSON-8-1 -> protovolt:TDSON-8-1
Changed lines of the file:
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@@
 			)
 		)
-		(property "Footprint" "Package_TO_SOT_SMD:TDSON-8-1"
+		(property "Footprint" "protovolt:TDSON-8-1"
 			(at 142.24 80.645 0)
 			(effects
@@
 			)
 		)
-		(property "Footprint" "Package_TO_SOT_SMD:TDSON-8-1"
+		(property "Footprint" "protovolt:TDSON-8-1"
 			(at 200.66 93.345 0)
 			(effects
@@
 			)
 		)
-		(property "Footprint" "Package_TO_SOT_SMD:TDSON-8-1"
+		(property "Footprint" "protovolt:TDSON-8-1"
 			(at 200.66 80.645 0)
 			(effects
@@
 			)
 		)
-		(property "Footprint" "Package_TO_SOT_SMD:TDSON-8-1"
+		(property "Footprint" "protovolt:TDSON-8-1"
 			(at 142.24 93.345 0)
 			(effects
@@
 			)
 		)
-		(property "Footprint" "Package_TO_SOT_SMD:TDSON-8-1"
+		(property "Footprint" "protovolt:TDSON-8-1"
 			(at 299.085 67.31 0)
 			(effects

Commit message: replace parts
Parts:
- removed C10: 39u 50V, Capacitor_SMD:CP_Elec_8x11.9, symbol Device:C_Polarized
- removed C4: 10u 100V, Capacitor_SMD:C_1210_3225Metric, symbol Device:C
- added NT1: NetTie_2, NetTie:NetTie-2_SMD_Pad0.5mm, symbol Device:NetTie_2
- C1: value 10u 100V -> 10u 50V; footprint Capacitor_SMD:C_1210_3225Metric -> Capacitor_SMD:C_0805_2012Metric; LCSC C5156756 -> C440198
- C11, C12, C13, C21: footprint Resistor_SMD:R_0603_1608Metric -> Capacitor_SMD:C_0402_1005Metric; LCSC C88219 -> C162178
- C14, C15, C16, C17, C22: footprint Capacitor_SMD:C_0603_1608Metric -> Capacitor_SMD:C_0402_1005Metric; LCSC C30926 -> C77020
- C18, C23: footprint Capacitor_SMD:C_0603_1608Metric -> Capacitor_SMD:C_0402_1005Metric; LCSC C1630 -> C107030
- C19, C20: footprint Capacitor_SMD:C_0603_1608Metric -> Capacitor_SMD:C_0402_1005Metric; LCSC C84419 -> C3845593
- C6, C9: value 39u 50V -> 47u 63V; footprint Capacitor_SMD:CP_Elec_8x11.9 -> Capacitor_SMD:CP_Elec_8x10.5; LCSC C193240 -> C5246568
- D1: footprint Diode_SMD:D_SOD-123 -> Diode_SMD:D_SOD-523; LCSC C2104 -> C131800
- Q1, Q2, Q3, Q4, Q5: value BSC0702LS -> HSBB6054; footprint protovolt:TDSON-8-1 -> Package_SON:Diodes_PowerDI3333-8; LCSC C501503 -> C5341686
- R1: footprint Resistor_SMD:R_2512_6332Metric -> protovolt:R_2512_6332Metric_SHUNT
- R22: LCSC C21376 -> C47500
- R3: footprint Resistor_SMD:R_1206_3216Metric -> protovolt:R_2512_6332Metric_SHUNT
Connections:
- net GND: now also NT1.1; no longer C12.1, C13.2, C19.2, C21.1, C25.2, C26.2, C27.2, C28.2, C29.2, J2.3 (Pin_3), J3.3 (Pin_3), J5.3 (Pin_3), J6.3 (Pin_3), J7.3 (Pin_3), J8.3 (Pin_3), R25.2, R26.2, R27.2, R28.2, R7.1, U2.17 (AGND), U2.41 (GND)
- new net GNDA: C12.1, C13.2, C19.2, C21.1, C25.2, C26.2, C27.2, C28.2, C29.2, J2.3 (Pin_3), J3.3 (Pin_3), J5.3 (Pin_3), J6.3 (Pin_3), J7.3 (Pin_3), J8.3 (Pin_3), NT1.2, R25.2, R26.2, R27.2, R28.2, R7.1, U2.17 (AGND), U2.41 (GND)
Other:
- note added: "BSC0702LS 60V 84A 83W 2.7mΩ@10V,50A 2.3V 1 N-channel TDSON-8-EP(5x6) MOSFETs ROHS BSC028N06LS3 60V 100A 2.8mΩ@10V,50A 139W 2.2V 1 N-channel TDSON-8(5.2x5.9) MOSFETs ROHS IAUC60N04S6L030HATMA HALF-BRIDGE AGM612MBQ HALF-BRIDGE HYG090ND06LS1C2 HALF-BRIDGE"
- note removed: "BSC0702LS 60V 84A 83W 2.7mΩ@10V,50A 2.3V 1 N-channel TDSON-8-EP(5x6) MOSFETs ROHS BSC028N06LS3 60V 100A 2.8mΩ@10V,50A 139W 2.2V 1 N-channel TDSON-8(5.2x5.9) MOSFETs ROHS IAUC60N04S6L030HATMA HALF-BRIDGE"

Commit message: retrace all
Parts:
- NT1: footprint NetTie:NetTie-2_SMD_Pad0.5mm -> protovolt:NetTie-2_SMD_Pad10mil
Connections:
- net GND: no longer U2.28 (PGND)
- net GNDA: now also U2.28 (PGND)
Changed lines of the file:
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@@
 	)
 	(junction
+		(at 186.69 220.98)
+		(diameter 0)
+		(color 0 0 0 0)
+	)
+	(junction
 		(at 356.87 161.29)
 		(diameter 0)
@@
 	)
 	(junction
-		(at 186.69 220.98)
-		(diameter 0)
-		(color 0 0 0 0)
-	)
-	(junction
 		(at 279.4 69.85)
 		(diameter 0)
@@
 	(wire
 		(pts
+			(xy 186.69 228.6) (xy 186.69 231.14)
+		)
+		(stroke
+			(width 0)
+			(type default)
+		)
+	)
+	(wire
+		(pts
 			(xy 359.41 151.13) (xy 359.41 152.4)
 		)
@@
 	(wire
 		(pts
-			(xy 186.69 220.98) (xy 187.96 220.98)
-		)
-		(stroke
-			(width 0)
-			(type default)
-		)
-	)
-	(wire
-		(pts
 			(xy 170.18 85.09) (xy 175.26 85.09)
 		)
@@
 	(wire
 		(pts
-			(xy 186.69 220.98) (xy 186.69 231.14)
-		)
-		(stroke
-			(width 0)
-			(type default)
-		)
-	)
-	(wire
-		(pts
 			(xy 232.41 69.85) (xy 232.41 74.93)
 		)
@@
 	(wire
 		(pts
+			(xy 360.68 228.6) (xy 360.68 231.14)
+		)
+		(stroke
+			(width 0)
+			(type default)
+		)
+	)
+	(wire
+		(pts
 			(xy 342.9 151.13) (xy 350.52 151.13)
 		)
@@
 	(wire
 		(pts
+			(xy 186.69 220.98) (xy 186.69 223.52)
+		)
+		(stroke
+			(width 0)
+			(type default)
+		)
+	)
+	(wire
+		(pts
 			(xy 185.42 173.99) (xy 203.2 173.99)
 		)
@@
 	(wire
 		(pts
-			(xy 193.04 220.98) (xy 194.31 220.98)
+			(xy 186.69 220.98) (xy 194.31 220.98)
 		)
 		(stroke
@@
 	)
 	(symbol
+		(lib_id "Device:NetTie_2")
+		(at 186.69 226.06 90)
+		(unit 1)
+		(exclude_from_sim no)
+		(in_bom no)
+		(on_board yes)
+		(dnp no)
+		(fields_autoplaced yes)
+		(property "Reference" "NT1"
+			(at 187.96 224.7899 90)
+			(effects
+				(font
+					(size 1.27 1.27)
+				)
+				(justify right)
+			)
+		)
+		(property "Value" "NetTie_2"
+			(at 187.96 227.3299 90)
+			(effects
+				(font
+					(size 1.27 1.27)
+				)
+				(justify right)
+			)
+		)
+		(property "Footprint" "protovolt:NetTie-2_SMD_Pad10mil"
+			(at 186.69 226.06 0)
+			(effects
+				(font
+					(size 1.27 1.27)
+				)
+				(hide yes)
+			)
+		)
+		(property "Datasheet" "~"
+			(at 186.69 226.06 0)
+			(effects
+				(font
+					(size 1.27 1.27)
+				)
+				(hide yes)
+			)
+		)
+		(property "Description" "Net tie, 2 pins"
+			(at 186.69 226.06 0)
+			(effects
+				(font
+					(size 1.27 1.27)
+				)
+				(hide yes)
+			)
+		)
+		(pin "2"
+		)
+		(pin "1"
+		)
+		(instances
+			(project "protovolt"
+				(path "/ea7037dc-92a2-412b-b904-472cbab72219/4a270319-7ef6-4bc5-85c2-eebc7d78bfc0"
+					(reference "NT1")
+					(unit 1)
+				)
+			)
+		)
+	)
+	(symbol
 		(lib_id "power:PWR_FLAG")
 		(at 353.06 231.14 180)
@@
 	)
 	(symbol
+		(lib_id "power:GNDA")
+		(at 360.68 228.6 180)
+		(unit 1)
+		(exclude_from_sim no)
+		(in_bom yes)
+		(on_board yes)
+		(dnp no)
+		(fields_autoplaced yes)
+		(property "Reference" "#PWR029"
+			(at 360.68 222.25 0)
+			(effects
+				(font
+					(size 1.27 1.27)
+				)
+				(hide yes)
+			)
+		)
+		(property "Value" "GNDA"
+			(at 360.68 223.52 0)
+			(effects
+				(font
+					(size 1.27 1.27)
+				)
+			)
+		)
+		(property "Footprint" ""
+			(at 360.68 228.6 0)
+			(effects
+				(font
+					(size 1.27 1.27)
+				)
+				(hide yes)
+			)
+		)
+		(property "Datasheet" ""
+			(at 360.68 228.6 0)
+			(effects
+				(font
+					(size 1.27 1.27)
+				)
+				(hide yes)
+			)
+		)
+		(property "Description" "Power symbol creates a global label with name \"GNDA\" , analog ground"
+			(at 360.68 228.6 0)
+			(effects
+				(font
+					(size 1.27 1.27)
+				)
+				(hide yes)
+			)
+		)
+		(pin "1"
+		)
+		(instances
+			(project "protovolt"
+				(path "/ea7037dc-92a2-412b-b904-472cbab72219/4a270319-7ef6-4bc5-85c2-eebc7d78bfc0"
+					(reference "#PWR029")
+					(unit 1)
+				)
+			)
+		)
+	)
+	(symbol
 		(lib_id "Device:C")
 		(at 245.11 162.56 180)
@@
 	)
 	(symbol
+		(lib_id "power:PWR_FLAG")
+		(at 360.68 231.14 180)
+		(unit 1)
+		(exclude_from_sim no)
+		(in_bom yes)
+		(on_board yes)
+		(dnp no)
+		(fields_autoplaced yes)
+		(property "Reference" "#FLG04"
+			(at 360.68 233.045 0)
+			(effects
+				(font
+					(size 1.27 1.27)
+				)
+				(hide yes)
+			)
+		)
+		(property "Value" "PWR_FLAG"
+			(at 360.68 236.22 0)
+			(effects
+				(font
+					(size 1.27 1.27)
+				)
+			)
+		)
+		(property "Footprint" ""
+			(at 360.68 231.14 0)
+			(effects
+				(font
+					(size 1.27 1.27)
+				)
+				(hide yes)
+			)
+		)
+		(property "Datasheet" "~"
+			(at 360.68 231.14 0)
+			(effects
+				(font
+					(size 1.27 1.27)
+				)
+				(hide yes)
+			)
+		)
+		(property "Description" "Special symbol for telling ERC where power comes from"
+			(at 360.68 231.14 0)
+			(effects
+				(font
+					(size 1.27 1.27)
+				)
+				(hide yes)
+			)
+		)
+		(pin "1"
+		)
+		(instances
+			(project "protovolt"
+				(path "/ea7037dc-92a2-412b-b904-472cbab72219/4a270319-7ef6-4bc5-85c2-eebc7d78bfc0"
+					(reference "#FLG04")
+					(unit 1)
+				)
+			)
+		)
+	)
+	(symbol
 		(lib_id "Device:R")
 		(at 140.97 226.06 0)
@@
 					(unit 1)
 				)
-			)
-		)
-	)
-	(symbol
-		(lib_id "Device:NetTie_2")
-		(at 190.5 220.98 0)
-		(unit 1)
-		(exclude_from_sim no)
-		(in_bom no)
-		(on_board yes)
-		(dnp no)
-		(fields_autoplaced yes)
-		(property "Reference" "NT1"
-			(at 190.5 215.9 0)
-			(effects
-				(font
-					(size 1.27 1.27)
-				)
-			)
-		)
-		(property "Value" "NetTie_2"
-			(at 190.5 218.44 0)
-			(effects
-				(font
-					(size 1.27 1.27)
-				)
-			)
-		)
-		(property "Footprint" "NetTie:NetTie-2_SMD_Pad0.5mm"
-			(at 190.5 220.98 0)
-			(effects
-				(font
-					(size 1.27 1.27)
-				)
-				(hide yes)
-			)
-		)
-		(property "Datasheet" "~"
-			(at 190.5 220.98 0)
-			(effects
-				(font
-					(size 1.27 1.27)
-				)
-				(hide yes)
-			)
-		)
-		(property "Description" "Net tie, 2 pins"
-			(at 190.5 220.98 0)
-			(effects
-				(font
-					(size 1.27 1.27)
-				)
-				(hide yes)
-			)
-		)
-		(pin "2"
-		)
-		(pin "1"
-		)
-		(instances
-			(project ""
-				(path "/ea7037dc-92a2-412b-b904-472cbab72219/4a270319-7ef6-4bc5-85c2-eebc7d78bfc0"
-					(reference "NT1")
-					(unit 1)
-				)
