File: hardware/protovolt/output_A.kicad_sch (KiCad schematic)
At the start: 75 parts, among them J1 Conn_01x03, J10 Conn_02x03_Odd_Even, J2 Conn_01x03, J3 Conn_01x03, J4 Conn_01x03, J5 Conn_01x03, J6 Conn_01x03, J7 Conn_01x03, J8 Conn_01x03, J9 Conn_02x03_Odd_Even, Q1 HSBB6054, Q2 HSBB6054, Q3 HSBB6054, Q4 HSBB6054, Q5 HSBB6054, U1 INA226, U2 LM51772RHAR

Commit message: add basic parts
Parts:
- C14, C15, C16, C17, C22: LCSC C77020 -> C307331
- R10, R14, R21, R23: LCSC C25139 -> C25077
- R13, R27, R6, R7, R9: LCSC C21376 -> C17168
- R3: LCSC C326610 -> C5375459
- R4: LCSC C25138 -> C25076
Changed lines of the file:
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@@
 			)
 		)
-		(property "LCSC" "C77020"
+		(property "LCSC" "C307331"
 			(at 308.61 162.56 0)
 			(effects
@@
 			)
 		)
-		(property "LCSC" "C25138"
+		(property "LCSC" "C25076"
 			(at 297.18 85.09 0)
 			(effects
@@
 			)
 		)
-		(property "LCSC" "C77020"
+		(property "LCSC" "C307331"
 			(at 207.01 185.42 0)
 			(effects
@@
 			)
 		)
-		(property "LCSC" "C25139"
+		(property "LCSC" "C25077"
 			(at 304.8 166.37 0)
 			(effects
@@
 			)
 		)
-		(property "LCSC" "C77020"
+		(property "LCSC" "C307331"
 			(at 245.11 162.56 0)
 			(effects
@@
 			)
 		)
-		(property "LCSC" "C21376"
+		(property "LCSC" "C17168"
 			(at 140.97 226.06 0)
 			(effects
@@
 			)
 		)
-		(property "LCSC" "C21376"
+		(property "LCSC" "C17168"
 			(at 137.16 156.21 0)
 			(effects
@@
 			)
 		)
-		(property "LCSC" "C21376"
+		(property "LCSC" "C17168"
 			(at 170.18 148.59 0)
 			(effects
@@
 			)
 		)
-		(property "LCSC" "C25139"
+		(property "LCSC" "C25077"
 			(at 248.92 190.5 0)
 			(effects
@@
 			)
 		)
-		(property "LCSC" "C25139"
+		(property "LCSC" "C25077"
 			(at 304.8 158.75 0)
 			(effects
@@
 			)
 		)
-		(property "LCSC" "C25139"
+		(property "LCSC" "C25077"
 			(at 248.92 198.12 0)
 			(effects
@@
 			)
 		)
-		(property "LCSC" "C77020"
+		(property "LCSC" "C307331"
 			(at 207.01 173.99 0)
 			(effects
@@
 			)
 		)
-		(property "LCSC" "C21376"
+		(property "LCSC" "C17168"
 			(at 248.92 166.37 0)
 			(effects
@@
 			)
 		)
-		(property "LCSC" "C21376"
+		(property "LCSC" "C17168"
 			(at 248.92 158.75 0)
 			(effects
@@
 			)
 		)
-		(property "LCSC" "C77020"
+		(property "LCSC" "C307331"
 			(at 336.55 144.78 0)
 			(effects
@@
 			)
 		)
-		(property "LCSC" "C326610 "
+		(property "LCSC" "C5375459"
 			(at 166.37 85.09 0)
 			(effects
