File: hardware/mini/mcu.kicad_sch (KiCad schematic)
At the start: 36 parts, among them U5 RP2040, U6 W25Q128JVP, Y1 12 MHz ABM8-272-T3

Commit message: cleanup schematic
Other:
- title: (none) -> Protovolt MINI
Changed lines of the file:
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@@
 	(generator_version "9.0")
 	(paper "A4")
+	(title_block
+		(title "Protovolt MINI")
+		(date "2025-06-16")
+		(rev "A")
+		(comment 3 "MINI")
+		(comment 4 "Protovolt")
+	)
 	(text "TPS55289 ENABLE"
 		(exclude_from_sim no)

Commit message: first fab run
Parts:
- removed TP5: P28, TestPoint:TestPoint_Pad_D1.0mm, symbol Connector:TestPoint
- added TP1: P29, TestPoint:TestPoint_Pad_D1.0mm, symbol Connector:TestPoint
- R18, R19, R20, R21, R22, R23, R24, R51: value 5.1k -> 4.7k; LCSC C25905 -> C25900
- R41: LCSC C25905 -> C25744
Connections:
- net P28 is gone; now on net DISP_RST: U5.40 (GPIO28_ADC2)
- net DISP_RST: no longer U5.31 (GPIO20)
- new net P20: TP1.1, U5.31 (GPIO20)
Changed lines of the file:
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@@
 	(wire
 		(pts
-			(xy 218.44 153.67) (xy 226.06 153.67)
-		)
-		(stroke
-			(width 0)
-			(type default)
-		)
-	)
-	(wire
-		(pts
 			(xy 157.48 138.43) (xy 157.48 140.97)
 		)
@@
 	(wire
 		(pts
-			(xy 118.11 158.75) (xy 123.19 158.75)
+			(xy 118.11 158.75) (xy 128.27 158.75)
 		)
 		(stroke
@@
 	(wire
 		(pts
+			(xy 218.44 153.67) (xy 226.06 153.67)
+		)
+		(stroke
+			(width 0)
+			(type default)
+		)
+	)
+	(wire
+		(pts
 			(xy 118.11 110.49) (xy 132.08 110.49)
 		)
@@
 	(wire
 		(pts
-			(xy 118.11 135.89) (xy 128.27 135.89)
+			(xy 118.11 135.89) (xy 123.19 135.89)
 		)
 		(stroke
@@
 		)
 	)
+	(label "P20"
+		(at 218.44 153.67 0)
+		(effects
+			(font
+				(size 1.27 1.27)
+			)
+			(justify left bottom)
+		)
+	)
 	(label "QSPI_SCLK"
 		(at 55.88 118.11 0)
@@
 		)
 	)
-	(label "P28"
-		(at 218.44 153.67 0)
+	(label "P20"
+		(at 123.19 135.89 180)
 		(effects
 			(font
 				(size 1.27 1.27)
 			)
-			(justify left bottom)
+			(justify right bottom)
 		)
 	)
@@
 		)
 	)
-	(label "P28"
-		(at 123.19 158.75 180)
-		(effects
-			(font
-				(size 1.27 1.27)
-			)
-			(justify right bottom)
-		)
-	)
 	(label "QSPI_SS"
 		(at 55.88 102.87 0)
@@
 		)
 	)
-	(hierarchical_label "DISP_RST"
-		(shape output)
-		(at 128.27 135.89 0)
-		(effects
-			(font
-				(size 1.27 1.27)
-			)
-			(justify left)
-		)
-	)
 	(hierarchical_label "USB_GPIO"
 		(shape input)
@@
 		)
 	)
+	(hierarchical_label "DISP_RST"
+		(shape output)
+		(at 128.27 158.75 0)
+		(effects
+			(font
+				(size 1.27 1.27)
+			)
+			(justify left)
+		)
+	)
 	(hierarchical_label "SENS_INT_A"
 		(shape input)
@@
 			)
 		)
-		(property "Value" "5.1k"
+		(property "Value" "4.7k"
 			(at 162.814 84.074 0)
 			(effects
@@
 			)
 		)
-		(property "LCSC" "C25905"
+		(property "LCSC" "C25900"
 			(at 162.56 78.74 0)
 			(effects
@@
 			)
 		)
-		(property "LCSC" "C25905"
+		(property "LCSC" "C25744"
 			(at 229.87 52.07 0)
 			(effects
@@
 	)
 	(symbol
+		(lib_id "Connector:TestPoint")
+		(at 226.06 153.67 270)
+		(unit 1)
+		(exclude_from_sim no)
+		(in_bom yes)
+		(on_board yes)
+		(dnp no)
+		(property "Reference" "TP1"
+			(at 231.14 152.146 90)
+			(effects
+				(font
+					(size 1.27 1.27)
+				)
+				(justify left)
+			)
+		)
+		(property "Value" "P29"
+			(at 231.14 154.432 90)
+			(effects
+				(font
+					(size 1.27 1.27)
+				)
+				(justify left)
+			)
+		)
+		(property "Footprint" "TestPoint:TestPoint_Pad_D1.0mm"
+			(at 226.06 158.75 0)
+			(effects
+				(font
+					(size 1.27 1.27)
+				)
+				(hide yes)
+			)
+		)
+		(property "Datasheet" "~"
+			(at 226.06 158.75 0)
+			(effects
+				(font
+					(size 1.27 1.27)
+				)
+				(hide yes)
+			)
+		)
+		(property "Description" "test point"
+			(at 226.06 153.67 0)
+			(effects
+				(font
+					(size 1.27 1.27)
+				)
+				(hide yes)
+			)
+		)
+		(pin "1"
+		)
+		(instances
+			(project "mini"
+				(path "/5aaaac9a-5acd-4aef-ad51-a6d04aa88705/8fbd1251-7beb-4aac-9406-53fe608f326c"
+					(reference "TP1")
+					(unit 1)
+				)
+			)
+		)
+	)
+	(symbol
 		(lib_id "Device:R")
 		(at 62.23 92.71 90)
@@
 			)
 		)
-		(property "Value" "5.1k"
+		(property "Value" "4.7k"
 			(at 157.734 84.074 0)
 			(effects
@@
 			)
 		)
-		(property "LCSC" "C25905"
+		(property "LCSC" "C25900"
 			(at 157.48 78.74 0)
 			(effects
@@
 			)
 		)
-		(property "Value" "5.1k"
+		(property "Value" "4.7k"
 			(at 147.828 84.074 0)
 			(effects
@@
 			)
 		)
-		(property "LCSC" "C25905"
+		(property "LCSC" "C25900"
 			(at 147.32 78.74 0)
 			(effects
@@
 			)
 		)
-		(property "Value" "5.1k"
+		(property "Value" "4.7k"
 			(at 152.654 84.074 0)
 			(effects
@@
 			)
 		)
-		(property "LCSC" "C25905"
+		(property "LCSC" "C25900"
 			(at 152.4 78.74 0)
 			(effects
@@
 			)
 		)
-		(property "Value" "5.1k"
+		(property "Value" "4.7k"
 			(at 157.988 139.954 0)
 			(effects
@@
 			)
 		)
-		(property "LCSC" "C25905"
+		(property "LCSC" "C25900"
 			(at 157.48 134.62 0)
 			(effects
@@
 			)
 		)
-		(property "Value" "5.1k"
+		(property "Value" "4.7k"
 			(at 162.814 139.954 0)
 			(effects
@@
 			)
 		)
-		(property "LCSC" "C25905"
+		(property "LCSC" "C25900"
 			(at 162.56 134.62 0)
 			(effects
@@
 	)
 	(symbol
-		(lib_id "Connector:TestPoint")
-		(at 226.06 153.67 270)
-		(unit 1)
-		(exclude_from_sim no)
-		(in_bom yes)
-		(on_board yes)
-		(dnp no)
-		(property "Reference" "TP5"
-			(at 231.14 152.146 90)
-			(effects
-				(font
-					(size 1.27 1.27)
-				)
-				(justify left)
-			)
-		)
-		(property "Value" "P28"
-			(at 231.14 154.432 90)
-			(effects
-				(font
-					(size 1.27 1.27)
-				)
-				(justify left)
-			)
-		)
-		(property "Footprint" "TestPoint:TestPoint_Pad_D1.0mm"
-			(at 226.06 158.75 0)
-			(effects
-				(font
-					(size 1.27 1.27)
-				)
-				(hide yes)
-			)
-		)
-		(property "Datasheet" "~"
-			(at 226.06 158.75 0)
-			(effects
-				(font
-					(size 1.27 1.27)
-				)
-				(hide yes)
-			)
-		)
-		(property "Description" "test point"
-			(at 226.06 153.67 0)
-			(effects
-				(font
-					(size 1.27 1.27)
-				)
-				(hide yes)
-			)
-		)
-		(pin "1"
-		)
-		(instances
-			(project "mini"
-				(path "/5aaaac9a-5acd-4aef-ad51-a6d04aa88705/8fbd1251-7beb-4aac-9406-53fe608f326c"
-					(reference "TP5")
-					(unit 1)
-				)
-			)
-		)
-	)
-	(symbol
 		(lib_id "power:GND")
 		(at 77.47 68.58 0)
@@
 			)
 		)
-		(property "Value" "5.1k"
+		(property "Value" "4.7k"
 			(at 152.654 114.554 0)
 			(effects
@@
 			)
 		)
-		(property "LCSC" "C25905"
+		(property "LCSC" "C25900"
 			(at 152.4 109.22 0)
 			(effects
@@
 			)
 		)
-		(property "Value" "5.1k"
+		(property "Value" "4.7k"
 			(at 147.828 114.554 0)
 			(effects
@@
 			)
 		)
-		(property "LCSC" "C25905"
+		(property "LCSC" "C25900"
 			(at 147.32 109.22 0)
 			(effects
