File: hardware/mini/power.kicad_sch (KiCad schematic)
At the start: 39 parts, among them U1 INA226, U2 TPS55289

Commit message: first fab run
Parts:
- R5: LCSC C25905 -> C25744
Changed lines of the file:
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@@
 			)
 		)
-		(property "LCSC" "C25905"
+		(property "LCSC" "C25744"
 			(at 158.75 151.13 0)
 			(effects
