File: hardware/mini/regulation.kicad_sch (KiCad schematic)
At the start: 11 parts, among them U4 TPS54202DDC

Commit message: first fab run
Parts:
- C27: value 56p -> 47p; LCSC C107007 -> C1567
- R11: now not fitted
Changed lines of the file:
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@@
 			)
 		)
-		(property "Value" "56p"
+		(property "Value" "47p"
 			(at 176.53 97.282 0)
 			(effects
@@
 			)
 		)
-		(property "LCSC" "C107007"
+		(property "LCSC" "C1567"
 			(at 181.61 96.52 0)
 			(effects
@@
 		(in_bom yes)
 		(on_board yes)
-		(dnp no)
+		(dnp yes)
 		(property "Reference" "R11"
 			(at 117.602 95.504 90)
